File: PCB/Audio_watermark_generator.kicad_sch (KiCad schematic)
At the start: 0 parts

Commit message: Refactor code structure for improved readability and maintainability
Parts:
- added C1, C4, C5: 1000nF, Capacitor_SMD:C_0805_2012Metric_Pad1.18x1.45mm_HandSolder, symbol Device:C
- added C2, C3: 3.3nF, Capacitor_SMD:C_0805_2012Metric_Pad1.18x1.45mm_HandSolder, symbol Device:C
- added R1: 3300R, Resistor_SMD:R_0805_2012Metric_Pad1.20x1.40mm_HandSolder, symbol Device:R
- added R10: 500000R, Resistor_SMD:R_0805_2012Metric_Pad1.20x1.40mm_HandSolder, symbol Device:R
- added R11, R12, R2, R3: 10000R, Resistor_SMD:R_0805_2012Metric_Pad1.20x1.40mm_HandSolder, symbol Device:R
- added R13, R16, R6, R8: 1000R, Resistor_SMD:R_0805_2012Metric_Pad1.20x1.40mm_HandSolder, symbol Device:R
- added R14, R15, R17: 330R, Resistor_SMD:R_0805_2012Metric_Pad1.20x1.40mm_HandSolder, symbol Device:R
- added R4, R5: 100000R, Resistor_SMD:R_0805_2012Metric_Pad1.20x1.40mm_HandSolder, symbol Device:R
- added R7: 1000000R, Resistor_SMD:R_0805_2012Metric_Pad1.20x1.40mm_HandSolder, symbol Device:R
- added R9: 10000000R, Resistor_SMD:R_0805_2012Metric_Pad1.20x1.40mm_HandSolder, symbol Device:R
- added SW1: SW_Push_DPDT, symbol Switch:SW_Push_DPDT
- added U1: STM32G431KBTx, Package_QFP:LQFP-32_7x7mm_P0.8mm, symbol MCU_ST_STM32G4:STM32G431KBTx
- added U2, U3, U5, U6, U7, U8, U9: TL072, symbol Amplifier_Operational:TL072
- added U4: PAM8303, Package_TO_SOT_SMD:SOT-23-6, symbol Amplifier_Audio:PAM8303
Connections:
- new net: R10.2, R9.1, U3.2 (-)
- new net: R9.2, U1.9 (PA4), U5.3 (+)
- new net: C3.1, R10.1, U3.1
- new net: U2.3 (+), U3.3 (+), U6.3 (+), U7.1, U7.2 (-)
- new net: R7.2, U5.1, U5.2 (-)
- new net: R14.1, R17.2, U8.1
- new net: U1.10 (PA5), U8.2 (-)
- new net: R13.2, R14.2, U8.3 (+)
- new net: R6.1, R7.1, R8.2, U6.2 (-)
- new net: R15.1, R17.1, U9.1
- new net: R3.1, R6.2, U2.1
- new net: C1.1, R1.2, SW1.6 (C)
- new net: C1.2, R2.2
- new net: R8.1, SW1.3 (C), U6.1
- new net: R11.1, U4.3 (IN)
- new net: R12.1, U4.4 (IN-)
- new net: U1.12 (PA7), U4.6 (EN)
- new net: R4.2, R5.1, U7.3 (+)
- new net: SW1.1 (A), SW1.4 (A)
- new net: R2.1, R3.2, U2.2 (-)
- new net: R15.2, R16.1, U9.3 (+)
- new net: C2.2, R12.2
- new net: C3.2, R11.2
- new net: U1.11 (PA6), U9.2 (-)
- new net: U1.16 (VSS), U1.32 (VSS)
- new net +3.3V: C4.2, C5.1, R1.1, R4.1, U4.5 (VDD), U4.7 (PVDD)
- new net GND: C2.1, C4.1, C5.2, R13.1, R16.2, R5.2, U4.2 (GND)

Commit message: Add DS3231 RTC component and power symbols to the schematic
Parts:
- added U10: ~, Connector_PinHeader_2.54mm:PinHeader_1x06_P2.54mm_Horizontal, symbol Timer_RTC:DS3231_TH
Connections:
- net +3.3V: now also U10.5 (VCC)
- net GND: now also U10.6 (GND)
- net at U1.18 (PA8): now also U10.4 (SDA)
- net at U1.19 (PA9): now also U10.3 (SCL)

Commit message: Final PCB design with all files included
Parts:
- removed C1, C4, C5: 1000nF, Capacitor_SMD:C_0805_2012Metric_Pad1.18x1.45mm_HandSolder, symbol Device:C
- removed C2, C3: 3.3nF, Capacitor_SMD:C_0805_2012Metric_Pad1.18x1.45mm_HandSolder, symbol Device:C
- removed R1: 3300R, Resistor_SMD:R_0805_2012Metric_Pad1.20x1.40mm_HandSolder, symbol Device:R
- removed R10: 500000R, Resistor_SMD:R_0805_2012Metric_Pad1.20x1.40mm_HandSolder, symbol Device:R
- removed R11, R12, R2, R3: 10000R, Resistor_SMD:R_0805_2012Metric_Pad1.20x1.40mm_HandSolder, symbol Device:R
- removed R13, R16, R6, R8: 1000R, Resistor_SMD:R_0805_2012Metric_Pad1.20x1.40mm_HandSolder, symbol Device:R
- removed R14, R15, R17: 330R, Resistor_SMD:R_0805_2012Metric_Pad1.20x1.40mm_HandSolder, symbol Device:R
- removed R4, R5: 100000R, Resistor_SMD:R_0805_2012Metric_Pad1.20x1.40mm_HandSolder, symbol Device:R
- removed R7: 1000000R, Resistor_SMD:R_0805_2012Metric_Pad1.20x1.40mm_HandSolder, symbol Device:R
- removed R9: 10000000R, Resistor_SMD:R_0805_2012Metric_Pad1.20x1.40mm_HandSolder, symbol Device:R
- removed SW1: SW_Push_DPDT, symbol Switch:SW_Push_DPDT
- removed U1: STM32G431KBTx, Package_QFP:LQFP-32_7x7mm_P0.8mm, symbol MCU_ST_STM32G4:STM32G431KBTx
- removed U10: ~, Connector_PinHeader_2.54mm:PinHeader_1x06_P2.54mm_Horizontal, symbol Timer_RTC:DS3231_TH
- removed U2, U3, U5, U6, U7, U8, U9: TL072, symbol Amplifier_Operational:TL072
- removed U4: PAM8303, Package_TO_SOT_SMD:SOT-23-6, symbol Amplifier_Audio:PAM8303
Other:
- added sheet Battery (battery.kicad_sch)
- added sheet Mixer (Mixer.kicad_sch)
- added sheet RTC (RTC.kicad_sch)
- added sheet STM32 (STM32.kicad_sch)
- added sheet Speaker (Speaker.kicad_sch)
- added sheet Transceiver (Transceiver.kicad_sch)
- company: (none) -> NTNU
- title: (none) -> CHIRP-SYNC - Audio Synchronization Module
